File: Zigbee Design/PCB Design/NXP_Smart_Charger.brd (EAGLE design)
At the start: 108.3 x 63.3 mm, 92 parts, among them IC1 MID400, IC2 MID400, IC3 LMV358, IC4 LMV358, Q1 2222A, Q2 2222A

Commit message: Add files via upload
Routing:
- net AC_TEST_2: track 4.33 -> 111.6 mm, vias 0 -> 1
- net AC_TEST: track 2.91 -> 101.9 mm, vias 0 -> 3
- net MOSI: track 0.00 -> 55.1 mm, vias 0 -> 1
- net SPI_CLK: track 0.00 -> 51.7 mm
- net PWM: track 0.00 -> 51.7 mm, vias 0 -> 5
- net MISO: track 0.00 -> 48.6 mm
- net SS: track 0.00 -> 45.1 mm
- net FORCE_START: track 3.87 -> 24.6 mm, vias 0 -> 1
- net PILOTREAD: track 66.0 -> 47.2 mm
- net BUTTON3: track 3.91 -> 21.8 mm, vias 0 -> 1
- net FORCE_STOP: track 3.89 -> 21.3 mm, vias 0 -> 1
- net 3.3V: track 56.1 -> 39.0 mm, vias 2 -> 4
- net GFCI_INT: track 55.2 -> 44.6 mm
- net +12V: track 71.0 -> 72.9 mm
- added copper zone on layer 1, net 3.3V
