File: Smartenit PCB/Smartenit_Board.sch (EAGLE design)
At the start: 86 parts, among them J1 2X5CONNECTOR1.27MM, Q1 QUARTZ_3.58M_2PIN, U1 SN74LVC1G3157, U2 ADE7953, U3 ESP-WROOM-32

Commit message: New Revision with grounds connected
Connections:
- net AGND: now also U3.GND@1, U3.GND@38; no longer U2.PAD
- net DGND: now also U2.PAD; no longer U3.GND@1, U3.GND@38
Changed lines of the file:
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@@
 <grid distance="0.1" unitdist="inch" unit="inch" style="lines" multiple="1" display="no" altdistance="0.01" altunitdist="inch" altunit="inch"/>
 <layers>
-<layer number="1" name="Top" color="4" fill="1" visible="yes" active="no"/>
-<layer number="2" name="Route2" color="1" fill="3" visible="yes" active="no"/>
-<layer number="3" name="Route3" color="4" fill="3" visible="yes" active="no"/>
-<layer number="4" name="Route4" color="1" fill="4" visible="yes" active="no"/>
-<layer number="5" name="Route5" color="4" fill="4" visible="yes" active="no"/>
-<layer number="6" name="Route6" color="1" fill="8" visible="yes" active="no"/>
-<layer number="7" name="Route7" color="4" fill="8" visible="yes" active="no"/>
-<layer number="8" name="Route8" color="1" fill="2" visible="yes" active="no"/>
-<layer number="9" name="Route9" color="4" fill="2" visible="yes" active="no"/>
-<layer number="10" name="Route10" color="1" fill="7" visible="yes" active="no"/>
-<layer number="11" name="Route11" color="4" fill="7" visible="yes" active="no"/>
-<layer number="12" name="Route12" color="1" fill="5" visible="yes" active="no"/>
-<layer number="13" name="Route13" color="4" fill="5" visible="yes" active="no"/>
-<layer number="14" name="Route14" color="1" fill="6" visible="yes" active="no"/>
-<layer number="15" name="Route15" color="4" fill="6" visible="yes" active="no"/>
-<layer number="16" name="Bottom" color="1" fill="1" visible="yes" active="no"/>
-<layer number="17" name="Pads" color="2" fill="1" visible="yes" active="no"/>
-<layer number="18" name="Vias" color="2" fill="1" visible="yes" active="no"/>
-<layer number="19" name="Unrouted" color="6" fill="1" visible="yes" active="no"/>
-<layer number="20" name="Dimension" color="15" fill="1" visible="yes" active="no"/>
-<layer number="21" name="tPlace" color="7" fill="1" visible="yes" active="no"/>
-<layer number="22" name="bPlace" color="7" fill="1" visible="yes" active="no"/>
-<layer number="23" name="tOrigins" color="15" fill="1" visible="yes" active="no"/>
-<layer number="24" name="bOrigins" color="15" fill="1" visible="yes" active="no"/>
-<layer number="25" name="tNames" color="7" fill="1" visible="yes" active="no"/>
-<layer number="26" name="bNames" color="7" fill="1" visible="yes" active="no"/>
-<layer number="27" name="tValues" color="7" fill="1" visible="yes" active="no"/>
-<layer number="28" name="bValues" color="7" fill="1" visible="yes" active="no"/>
+<layer number="1" name="Top" color="4" fill="1" visible="no" active="no"/>
+<layer number="2" name="Route2" color="1" fill="3" visible="no" active="no"/>
+<layer number="3" name="Route3" color="4" fill="3" visible="no" active="no"/>
+<layer number="4" name="Route4" color="1" fill="4" visible="no" active="no"/>
+<layer number="5" name="Route5" color="4" fill="4" visible="no" active="no"/>
+<layer number="6" name="Route6" color="1" fill="8" visible="no" active="no"/>
+<layer number="7" name="Route7" color="4" fill="8" visible="no" active="no"/>
+<layer number="8" name="Route8" color="1" fill="2" visible="no" active="no"/>
+<layer number="9" name="Route9" color="4" fill="2" visible="no" active="no"/>
+<layer number="10" name="Route10" color="1" fill="7" visible="no" active="no"/>
+<layer number="11" name="Route11" color="4" fill="7" visible="no" active="no"/>
+<layer number="12" name="Route12" color="1" fill="5" visible="no" active="no"/>
+<layer number="13" name="Route13" color="4" fill="5" visible="no" active="no"/>
+<layer number="14" name="Route14" color="1" fill="6" visible="no" active="no"/>
+<layer number="15" name="Route15" color="4" fill="6" visible="no" active="no"/>
+<layer number="16" name="Bottom" color="1" fill="1" visible="no" active="no"/>
+<layer number="17" name="Pads" color="2" fill="1" visible="no" active="no"/>
+<layer number="18" name="Vias" color="2" fill="1" visible="no" active="no"/>
+<layer number="19" name="Unrouted" color="6" fill="1" visible="no" active="no"/>
+<layer number="20" name="Dimension" color="15" fill="1" visible="no" active="no"/>
+<layer number="21" name="tPlace" color="7" fill="1" visible="no" active="no"/>
+<layer number="22" name="bPlace" color="7" fill="1" visible="no" active="no"/>
+<layer number="23" name="tOrigins" color="15" fill="1" visible="no" active="no"/>
+<layer number="24" name="bOrigins" color="15" fill="1" visible="no" active="no"/>
+<layer number="25" name="tNames" color="7" fill="1" visible="no" active="no"/>
+<layer number="26" name="bNames" color="7" fill="1" visible="no" active="no"/>
+<layer number="27" name="tValues" color="7" fill="1" visible="no" active="no"/>
+<layer number="28" name="bValues" color="7" fill="1" visible="no" active="no"/>
 <layer number="29" name="tStop" color="7" fill="3" visible="no" active="no"/>
 <layer number="30" name="bStop" color="7" fill="6" visible="no" active="no"/>
@@
 <layer number="35" name="tGlue" color="7" fill="4" visible="no" active="no"/>
 <layer number="36" name="bGlue" color="7" fill="5" visible="no" active="no"/>
-<layer number="37" name="tTest" color="7" fill="1" visible="yes" active="no"/>
-<layer number="38" name="bTest" color="7" fill="1" visible="yes" active="no"/>
+<layer number="37" name="tTest" color="7" fill="1" visible="no" active="no"/>
+<layer number="38" name="bTest" color="7" fill="1" visible="no" active="no"/>
 <layer number="39" name="tKeepout" color="4" fill="11" visible="no" active="no"/>
 <layer number="40" name="bKeepout" color="1" fill="11" visible="no" active="no"/>
@@
 <layer number="44" name="Drills" color="7" fill="1" visible="no" active="no"/>
 <layer number="45" name="Holes" color="7" fill="1" visible="no" active="no"/>
-<layer number="46" name="Milling" color="3" fill="1" visible="yes" active="no"/>
-<layer number="47" name="Measures" color="7" fill="1" visible="yes" active="no"/>
-<layer number="48" name="Document" color="7" fill="1" visible="yes" active="no"/>
-<layer number="49" name="Reference" color="14" fill="1" visible="yes" active="no"/>
-<layer number="50" name="dxf" color="7" fill="1" visible="yes" active="no"/>
-<layer number="51" name="tDocu" color="6" fill="1" visible="yes" active="no"/>
-<layer number="52" name="bDocu" color="6" fill="1" visible="yes" active="no"/>
-<layer number="53" name="tGND_GNDA" color="7" fill="9" visible="yes" active="no"/>
-<layer number="54" name="bGND_GNDA" color="1" fill="9" visible="yes" active="no"/>
-<layer number="56" name="wert" color="7" fill="1" visible="yes" active="no"/>
-<layer number="57" name="tCAD" color="7" fill="1" visible="yes" active="no"/>
-<layer number="59" name="tCarbon" color="7" fill="1" visible="yes" active="no"/>
-<layer number="60" name="bCarbon" color="7" fill="1" visible="yes" active="no"/>
+<layer number="46" name="Milling" color="3" fill="1" visible="no" active="no"/>
+<layer number="47" name="Measures" color="7" fill="1" visible="no" active="no"/>
+<layer number="48" name="Document" color="7" fill="1" visible="no" active="no"/>
+<layer number="49" name="Reference" color="14" fill="1" visible="no" active="no"/>
+<layer number="50" name="dxf" color="7" fill="1" visible="no" active="no"/>
+<layer number="51" name="tDocu" color="6" fill="1" visible="no" active="no"/>
+<layer number="52" name="bDocu" color="6" fill="1" visible="no" active="no"/>
+<layer number="53" name="tGND_GNDA" color="7" fill="9" visible="no" active="no"/>
+<layer number="54" name="bGND_GNDA" color="1" fill="9" visible="no" active="no"/>
+<layer number="56" name="wert" color="7" fill="1" visible="no" active="no"/>
+<layer number="57" name="tCAD" color="7" fill="1" visible="no" active="no"/>
+<layer number="59" name="tCarbon" color="7" fill="1" visible="no" active="no"/>
+<layer number="60" name="bCarbon" color="7" fill="1" visible="no" active="no"/>
 <layer number="88" name="SimResults" color="9" fill="1" visible="no" active="yes"/>
 <layer number="89" name="SimProbes" color="9" fill="1" visible="no" active="yes"/>
@@
 </segment>
 <segment>
-<pinref part="U2" gate="G$1" pin="PAD"/>
-<pinref part="GNDI30" gate="1" pin="GND"/>
-<wire x1="-205.74" y1="-91.44" x2="-205.74" y2="-63.5" width="0.1524" layer="91"/>
-</segment>
-<segment>
 <pinref part="U3" gate="G$1" pin="GND"/>
 <pinref part="GND10" gate="1" pin="GND"/>
 <wire x1="-5.08" y1="53.34" x2="-5.08" y2="50.8" width="0.1524" layer="91"/>
+</segment>
+<segment>
+<pinref part="U3" gate="G$1" pin="GND@1"/>
+<pinref part="GND6" gate="1" pin="GND"/>
+<wire x1="-30.48" y1="73.66" x2="-38.1" y2="73.66" width="0.1524" layer="91"/>
+</segment>
+<segment>
+<pinref part="U3" gate="G$1" pin="GND@38"/>
+<pinref part="GND8" gate="1" pin="GND"/>
+<wire x1="17.78" y1="73.66" x2="22.86" y2="73.66" width="0.1524" layer="91"/>
 </segment>
 </net>
@@
 </segment>
 <segment>
-<pinref part="U3" gate="G$1" pin="GND@1"/>
-<pinref part="GND6" gate="1" pin="GND"/>
-<wire x1="-30.48" y1="73.66" x2="-38.1" y2="73.66" width="0.1524" layer="91"/>
-</segment>
-<segment>
-<pinref part="U3" gate="G$1" pin="GND@38"/>
-<pinref part="GND8" gate="1" pin="GND"/>
-<wire x1="17.78" y1="73.66" x2="22.86" y2="73.66" width="0.1524" layer="91"/>
-</segment>
-<segment>
 <pinref part="GNDI5" gate="1" pin="GND"/>
 <pinref part="R36" gate="G$1" pin="1"/>
@@
 <wire x1="-210.82" y1="-83.82" x2="-210.82" y2="-63.5" width="0.1524" layer="91"/>
 </segment>
-</net>
+<segment>
+<pinref part="U2" gate="G$1" pin="PAD"/>
+<pinref part="GNDI30" gate="1" pin="GND"/>
+<wire x1="-205.74" y1="-91.44" x2="-205.74" y2="-63.5" width="0.1524" layer="91"/>
+</segment>
+</net>

Commit message: Made Al's Revision Suggestions
-no right angles
-flipped header
-New digital ground plane (redid ground signals)
-Reorganized ADE7953 components
Connections:
- removed net N$10: C18.1, U2.I1N
- removed net N$13: C14.1, U2.I2N
- net AGND: now also C3.1, D1.A, J1.10, R15.1, R32.1, R34.1, R35.1, R36.1, S100.1, U$1.S1, U$4.GND; no longer C10.2, C11.2, C14.2, C17.1, C18.2, C19.2, C20.2, C4.1, R17.2, R19.2, R20.1, R21.1, R23.2, R24.2, R26.1, R29.1, R30.2, R31.2
- net DGND: now also C10.2, C11.2, C14.2, C17.1, C18.2, C19.2, C20.2, C4.1, R17.2, R19.2, R20.1, R21.1, R23.2, R24.2, R26.1, R29.1, R30.2, R31.2; no longer C3.1, D1.A, J1.10, R15.1, R32.1, R34.1, R35.1, R36.1, S100.1, U$1.S1, U$4.GND
- net N$11: now also C14.1, U2.I2N
- net N$27: now also C18.1, U2.I1N

Commit message: Additional Modifications from Al
-moved mplex to connector region
-fixed ground connections to match Als exactly
-additional reogranization of traces
Connections:
- net AGND: now also C10.2, C11.2, C12.1, C13.1, C14.2, C17.1, C18.2, C19.2, C20.2, C4.1, R17.2, R19.2, R20.1, R21.1, R23.2, R24.2, R26.1, R29.1, R30.2, R31.2; no longer C1.1, C2.2, C21.2, C22.-, C23.1, C24.-, C3.1, C5.1, C6.1, C7.1, C8.1, C9.1, D1.A, D2.A, D3.P, J1.10, R15.1, R2.1, R32.1, R34.1, R35.1, R36.1, S100.1, U$1.S1, U$4.GND, U$5.PIN5, U2.PULL_LOW, U3.GND, U3.GND@1, U3.GND@15, U3.GND@38
- net DGND: now also C1.1, C2.2, C21.2, C22.-, C23.1, C24.-, C3.1, C5.1, C6.1, C7.1, C8.1, C9.1, D1.A, D2.A, D3.P, J1.10, R15.1, R2.1, R32.1, R34.1, R35.1, R36.1, S100.1, U$1.S1, U$4.GND, U$5.PIN5, U2.PULL_LOW, U3.GND, U3.GND@1, U3.GND@15, U3.GND@38; no longer C10.2, C11.2, C12.1, C13.1, C14.2, C17.1, C18.2, C19.2, C20.2, C4.1, R17.2, R19.2, R20.1, R21.1, R23.2, R24.2, R26.1, R29.1, R30.2, R31.2
Changed lines of the file:
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@@
 </segment>
 </net>
-<net name="AGND" class="0">
-<segment>
-<pinref part="U2" gate="G$1" pin="AGND"/>
-<pinref part="GNDI19" gate="1" pin="GND"/>
-<wire x1="-213.36" y1="-66.04" x2="-213.36" y2="-63.5" width="0.1524" layer="91"/>
-</segment>
+<net name="DGND" class="0">
 <segment>
 <pinref part="C7" gate="G$1" pin="1"/>
@@
 </segment>
 <segment>
-<pinref part="U1" gate="G$1" pin="GND"/>
-<pinref part="GND12" gate="1" pin="GND"/>
-<wire x1="-287.02" y1="-83.82" x2="-292.1" y2="-83.82" width="0.1524" layer="91"/>
-</segment>
-<segment>
 <pinref part="GND4" gate="1" pin="GND"/>
 <pinref part="D2" gate="G$1" pin="A"/>
@@
 </segment>
 <segment>
-<wire x1="-322.58" y1="33.02" x2="-307.34" y2="33.02" width="0.1524" layer="91"/>
-<pinref part="GNDI16" gate="1" pin="GND"/>
-<wire x1="-307.34" y1="33.02" x2="-307.34" y2="30.48" width="0.1524" layer="91"/>
-<pinref part="U$3" gate="G$1" pin="7"/>
-</segment>
-<segment>
 <wire x1="-289.56" y1="38.1" x2="-271.78" y2="38.1" width="0.1524" layer="91"/>
 <pinref part="GNDI13" gate="1" pin="GND"/>
@@
 <wire x1="-15.24" y1="-58.42" x2="-15.24" y2="-55.88" width="0.1524" layer="91"/>
 </segment>
+<segment>
+<pinref part="U2" gate="G$1" pin="DGND"/>
+<pinref part="GNDI20" gate="1" pin="GND"/>
+<wire x1="-210.82" y1="-83.82" x2="-210.82" y2="-63.5" width="0.1524" layer="91"/>
+</segment>
+<segment>
+<pinref part="C16" gate="G$1" pin="1"/>
+<wire x1="-152.4" y1="-33.02" x2="-147.32" y2="-33.02" width="0.1524" layer="91"/>
+<pinref part="C15" gate="G$1" pin="1"/>
+<wire x1="-147.32" y1="-33.02" x2="-144.78" y2="-33.02" width="0.1524" layer="91"/>
+<junction x="-147.32" y="-33.02"/>
+<pinref part="GNDI17" gate="1" pin="GND"/>
+</segment>
+<segment>
+<pinref part="U2" gate="G$1" pin="PAD"/>
+<pinref part="GNDI30" gate="1" pin="GND"/>
+<wire x1="-205.74" y1="-91.44" x2="-205.74" y2="-63.5" width="0.1524" layer="91"/>
+</segment>
 </net>
-<net name="DGND" class="0">
+<net name="AGND" class="0">
 <segment>
 <pinref part="C13" gate="G$1" pin="1"/>
@@
 <junction x="-165.1" y="-35.56"/>
 <pinref part="GNDI18" gate="1" pin="GND"/>
-</segment>
-<segment>
-<pinref part="C16" gate="G$1" pin="1"/>
-<wire x1="-152.4" y1="-33.02" x2="-147.32" y2="-33.02" width="0.1524" layer="91"/>
-<pinref part="C15" gate="G$1" pin="1"/>
-<wire x1="-147.32" y1="-33.02" x2="-144.78" y2="-33.02" width="0.1524" layer="91"/>
-<junction x="-147.32" y="-33.02"/>
-<pinref part="GNDI17" gate="1" pin="GND"/>
-</segment>
-<segment>
-<pinref part="U2" gate="G$1" pin="DGND"/>
-<pinref part="GNDI20" gate="1" pin="GND"/>
-<wire x1="-210.82" y1="-83.82" x2="-210.82" y2="-63.5" width="0.1524" layer="91"/>
 </segment>
 <segment>
@@
 </segment>
 <segment>
-<pinref part="U2" gate="G$1" pin="PAD"/>
-<pinref part="GNDI30" gate="1" pin="GND"/>
-<wire x1="-205.74" y1="-91.44" x2="-205.74" y2="-63.5" width="0.1524" layer="91"/>
+<pinref part="U1" gate="G$1" pin="GND"/>
+<pinref part="GND12" gate="1" pin="GND"/>
+<wire x1="-287.02" y1="-83.82" x2="-292.1" y2="-83.82" width="0.1524" layer="91"/>
+</segment>
+<segment>
+<pinref part="U2" gate="G$1" pin="AGND"/>
+<pinref part="GNDI19" gate="1" pin="GND"/>
+<wire x1="-213.36" y1="-66.04" x2="-213.36" y2="-63.5" width="0.1524" layer="91"/>
+</segment>
+<segment>
+<wire x1="-322.58" y1="33.02" x2="-307.34" y2="33.02" width="0.1524" layer="91"/>
+<pinref part="GNDI16" gate="1" pin="GND"/>
+<wire x1="-307.34" y1="33.02" x2="-307.34" y2="30.48" width="0.1524" layer="91"/>
+<pinref part="U$3" gate="G$1" pin="7"/>
 </segment>
 </net>
