File: Smartenit PCB/Smartenit_Board.sch (EAGLE design)
At the start: 86 parts, among them J1 2X5CONNECTOR1.27MM, Q1 QUARTZ_3.58M_2PIN, U1 SN74LVC1G3157, U2 ADE7953, U3 ESP-WROOM-32

Commit message: fixed MPLEX package, reverses L1/L2 lines
Parts:
- R39: value 100k -> 10k
Connections:
- net DIO11 renamed RELAY1
- net DIO12 renamed RELAY2
- net GFI_TEST renamed RELAY_EN
- net SS renamed FRGGN
- removed net N$54: R13.2, U1.B2
- removed net N$55: R4.2, U1.B1
- new net N$10: R4.2, U1.B2
- new net N$13: R13.2, U1.B1
Other:
- moved on the sheet: R13, R4
Changed lines of the file:
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@@
 <part name="GNDI13" library="SparkFun" deviceset="GND" device=""/>
 <part name="GNDI16" library="SparkFun" deviceset="GND" device=""/>
-<part name="R39" library="SparkFun-Resistors" deviceset="100KOHM" device="-0603-1/10W-1%" value="100k"/>
+<part name="R39" library="SparkFun-Resistors" deviceset="100KOHM" device="-0603-1/10W-1%" value="10k"/>
 <part name="Q2" library="semicon-smd-ipc" library_urn="urn:adsk.eagle:library:353" deviceset="PNP-TRANSISTOR_" device="SOT23" package3d_urn="urn:adsk.eagle:package:26310/1"/>
 <part name="P+4" library="SparkFun" deviceset="3.3V" device=""/>
@@
 <instance part="U1" gate="G$1" x="-274.32" y="-83.82"/>
 <instance part="GND12" gate="1" x="-294.64" y="-83.82" rot="R270"/>
-<instance part="R13" gate="G$1" x="-302.26" y="-78.74"/>
-<instance part="R4" gate="G$1" x="-302.26" y="-88.9"/>
+<instance part="R13" gate="G$1" x="-302.26" y="-88.9"/>
+<instance part="R4" gate="G$1" x="-302.26" y="-78.74"/>
 <instance part="P+11" gate="G$1" x="-256.54" y="-83.82" rot="R270"/>
 <instance part="J1" gate="G$1" x="-71.12" y="-50.8"/>
@@
 <segment>
 <pinref part="R13" gate="G$1" pin="1"/>
-<wire x1="-307.34" y1="-78.74" x2="-320.04" y2="-78.74" width="0.1524" layer="91"/>
-<label x="-317.5" y="-78.74" size="1.778" layer="95"/>
+<wire x1="-307.34" y1="-88.9" x2="-320.04" y2="-88.9" width="0.1524" layer="91"/>
+<label x="-317.5" y="-88.9" size="1.778" layer="95"/>
 </segment>
 </net>
@@
 <segment>
 <pinref part="R4" gate="G$1" pin="1"/>
-<wire x1="-307.34" y1="-88.9" x2="-322.58" y2="-88.9" width="0.1524" layer="91"/>
-<label x="-317.5" y="-88.9" size="1.778" layer="95"/>
-</segment>
-</net>
-<net name="DIO12" class="0">
-<segment>
-<wire x1="-289.56" y1="43.18" x2="-276.86" y2="43.18" width="0.1524" layer="91"/>
-<label x="-287.02" y="43.18" size="1.778" layer="95"/>
-<pinref part="U$5" gate="G$1" pin="PIN3"/>
-</segment>
-<segment>
-<pinref part="U3" gate="G$1" pin="IO33"/>
-<wire x1="-30.48" y1="53.34" x2="-40.64" y2="53.34" width="0.1524" layer="91"/>
-<label x="-45.72" y="53.34" size="1.778" layer="95"/>
-</segment>
-</net>
-<net name="DIO11" class="0">
-<segment>
-<wire x1="-289.56" y1="45.72" x2="-276.86" y2="45.72" width="0.1524" layer="91"/>
-<label x="-287.02" y="45.72" size="1.778" layer="95"/>
-<pinref part="U$5" gate="G$1" pin="PIN2"/>
-</segment>
-<segment>
-<pinref part="U3" gate="G$1" pin="IO32"/>
-<wire x1="-30.48" y1="55.88" x2="-40.64" y2="55.88" width="0.1524" layer="91"/>
-<label x="-45.72" y="55.88" size="1.778" layer="95"/>
+<wire x1="-307.34" y1="-78.74" x2="-322.58" y2="-78.74" width="0.1524" layer="91"/>
+<label x="-317.5" y="-78.74" size="1.778" layer="95"/>
 </segment>
 </net>
@@
 <pinref part="Q2" gate="G$1" pin="C"/>
 <wire x1="-259.08" y1="48.26" x2="-259.08" y2="53.34" width="0.1524" layer="91"/>
-</segment>
-</net>
-<net name="GFI_TEST" class="0">
-<segment>
-<pinref part="Q2" gate="G$1" pin="B"/>
-<wire x1="-254" y1="58.42" x2="-243.84" y2="58.42" width="0.1524" layer="91"/>
-<label x="-248.92" y="58.42" size="1.778" layer="95"/>
-</segment>
-<segment>
-<pinref part="U3" gate="G$1" pin="IO21"/>
-<wire x1="17.78" y1="60.96" x2="27.94" y2="60.96" width="0.1524" layer="91"/>
-<label x="20.32" y="60.96" size="1.778" layer="95"/>
 </segment>
 </net>
@@
 </segment>
 </net>
-<net name="SS" class="0">
+<net name="FRGGN" class="0">
 <segment>
 <pinref part="U3" gate="G$1" pin="IO15"/>
 <wire x1="2.54" y1="30.48" x2="2.54" y2="20.32" width="0.1524" layer="91"/>
-<label x="2.54" y="20.32" size="1.778" layer="95" rot="R90"/>
 <pinref part="R32" gate="G$1" pin="2"/>
 </segment>
@@
 <pinref part="U3" gate="G$1" pin="SENSOR_VP"/>
 <wire x1="-30.48" y1="66.04" x2="-40.64" y2="66.04" width="0.1524" layer="91"/>
-</segment>
-</net>
-<net name="N$54" class="0">
-<segment>
-<pinref part="R13" gate="G$1" pin="2"/>
-<pinref part="U1" gate="G$1" pin="B2"/>
-<wire x1="-297.18" y1="-78.74" x2="-287.02" y2="-78.74" width="0.1524" layer="91"/>
-</segment>
-</net>
-<net name="N$55" class="0">
-<segment>
-<pinref part="R4" gate="G$1" pin="2"/>
-<pinref part="U1" gate="G$1" pin="B1"/>
-<wire x1="-297.18" y1="-88.9" x2="-287.02" y2="-88.9" width="0.1524" layer="91"/>
 </segment>
 </net>
@@
 </segment>
 </net>
+<net name="RELAY_EN" class="0">
+<segment>
+<pinref part="U3" gate="G$1" pin="IO21"/>
+<wire x1="17.78" y1="60.96" x2="27.94" y2="60.96" width="0.1524" layer="91"/>
+<label x="20.32" y="60.96" size="1.778" layer="95"/>
+</segment>
+<segment>
+<pinref part="Q2" gate="G$1" pin="B"/>
+<wire x1="-254" y1="58.42" x2="-243.84" y2="58.42" width="0.1524" layer="91"/>
+<label x="-248.92" y="58.42" size="1.778" layer="95"/>
+</segment>
+</net>
+<net name="RELAY1" class="0">
+<segment>
+<wire x1="-289.56" y1="45.72" x2="-276.86" y2="45.72" width="0.1524" layer="91"/>
+<label x="-287.02" y="45.72" size="1.778" layer="95"/>
+<pinref part="U$5" gate="G$1" pin="PIN2"/>
+</segment>
+<segment>
+<pinref part="U3" gate="G$1" pin="IO32"/>
+<wire x1="-30.48" y1="55.88" x2="-40.64" y2="55.88" width="0.1524" layer="91"/>
+<label x="-45.72" y="55.88" size="1.778" layer="95"/>
+</segment>
+</net>
+<net name="RELAY2" class="0">
+<segment>
+<wire x1="-289.56" y1="43.18" x2="-276.86" y2="43.18" width="0.1524" layer="91"/>
+<label x="-287.02" y="43.18" size="1.778" layer="95"/>
+<pinref part="U$5" gate="G$1" pin="PIN3"/>
+</segment>
+<segment>
+<pinref part="U3" gate="G$1" pin="IO33"/>
+<wire x1="-30.48" y1="53.34" x2="-40.64" y2="53.34" width="0.1524" layer="91"/>
+<label x="-45.72" y="53.34" size="1.778" layer="95"/>
+</segment>
+</net>
+<net name="N$10" class="0">
+<segment>
+<pinref part="R4" gate="G$1" pin="2"/>
+<pinref part="U1" gate="G$1" pin="B2"/>
+<wire x1="-297.18" y1="-78.74" x2="-287.02" y2="-78.74" width="0.1524" layer="91"/>
+</segment>
+</net>
+<net name="N$13" class="0">
+<segment>
+<pinref part="U1" gate="G$1" pin="B1"/>
+<pinref part="R13" gate="G$1" pin="2"/>
+<wire x1="-287.02" y1="-88.9" x2="-297.18" y2="-88.9" width="0.1524" layer="91"/>
+</segment>
+</net>

Commit message: stuff
Parts:
- added R43, R44: 4.7k, SparkFun-Resistors:1KOHM-0603-1/10W-1%
Connections:
- new net GND: R43.2, R44.1
- net N$10: now also R43.1
- net N$13: now also R44.2
Changed lines of the file:
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@@
 <part name="D3" library="Smart_Charger" deviceset="SS32_DIODE" device=""/>
 <part name="D1" library="Smart_Charger" deviceset="TVSDIODE" device="" value="P6SMB16A"/>
+<part name="R43" library="SparkFun-Resistors" deviceset="1KOHM" device="-0603-1/10W-1%" value="4.7k"/>
+<part name="R44" library="SparkFun-Resistors" deviceset="1KOHM" device="-0603-1/10W-1%" value="4.7k"/>
+<part name="DFGND" library="SparkFun" deviceset="GND" device=""/>
+<part name="DGND" library="SparkFun" deviceset="GND" device=""/>
 </parts>
 <sheets>
@@
 <attribute name="NAME" x="-221.4626" y="170.18" size="1.778" layer="95" rot="R90"/>
 </instance>
+<instance part="R43" gate="G$1" x="-292.1" y="-73.66" rot="R90"/>
+<instance part="R44" gate="G$1" x="-292.1" y="-96.52" rot="R90"/>
+<instance part="DFGND" gate="1" x="-292.1" y="-63.5" rot="R180"/>
+<instance part="DGND" gate="1" x="-292.1" y="-106.68"/>
 </instances>
 <busses>
@@
 <pinref part="R4" gate="G$1" pin="2"/>
 <pinref part="U1" gate="G$1" pin="B2"/>
-<wire x1="-297.18" y1="-78.74" x2="-287.02" y2="-78.74" width="0.1524" layer="91"/>
+<wire x1="-297.18" y1="-78.74" x2="-292.1" y2="-78.74" width="0.1524" layer="91"/>
+<pinref part="R43" gate="G$1" pin="1"/>
+<wire x1="-292.1" y1="-78.74" x2="-287.02" y2="-78.74" width="0.1524" layer="91"/>
+<junction x="-292.1" y="-78.74"/>
 </segment>
 </net>
@@
 <pinref part="U1" gate="G$1" pin="B1"/>
 <pinref part="R13" gate="G$1" pin="2"/>
-<wire x1="-287.02" y1="-88.9" x2="-297.18" y2="-88.9" width="0.1524" layer="91"/>
-</segment>
-</net>
+<wire x1="-287.02" y1="-88.9" x2="-292.1" y2="-88.9" width="0.1524" layer="91"/>
+<pinref part="R44" gate="G$1" pin="2"/>
+<wire x1="-292.1" y1="-88.9" x2="-297.18" y2="-88.9" width="0.1524" layer="91"/>
+<wire x1="-292.1" y1="-91.44" x2="-292.1" y2="-88.9" width="0.1524" layer="91"/>
+<junction x="-292.1" y="-88.9"/>
+</segment>
+</net>
+<net name="GND" class="0">
+<segment>
+<pinref part="R43" gate="G$1" pin="2"/>
+<pinref part="DFGND" gate="1" pin="GND"/>
+<wire x1="-292.1" y1="-68.58" x2="-292.1" y2="-66.04" width="0.1524" layer="91"/>
+</segment>
+<segment>
+<pinref part="R44" gate="G$1" pin="1"/>
+<pinref part="DGND" gate="1" pin="GND"/>
+<wire x1="-292.1" y1="-101.6" x2="-292.1" y2="-104.14" width="0.1524" layer="91"/>
+</segment>
+</net>
